File: S2020/PowerSupply.sch (KiCad schematic (older format))
At the start: 25 parts, among them T1 4:1

Commit message: test edit
Parts:
- removed D1: 1N4735A, symbol 00TJR:ZENER-RESCUE-F2018
- removed RL, Rs: 1kΩ, symbol S2020-rescue:R_US-sDevice
- added D?: 1N4735A, symbol 00TJR:ZENER-RESCUE-F2018
- added RL?: 1kΩ, symbol S2020-rescue:R_US-sDevice
- added Rs?: 1kΩ 2W, symbol S2020-rescue:R_US-sDevice
Connections:
- net GND: now also D?.2 (A), RL?.2
- new net: D?.1 (K), RL?.1, Rs?.2
Changed lines of the file:
@@
 EESchema Schematic File Version 4
-LIBS:S2020-cache
 EELAYER 30 0
 EELAYER END
@@
 $EndComp
 $Comp
-L S2020-rescue:R_US-sDevice RL
-U 1 1 5F2E19B9
-P 2200 3450
-F 0 "RL" H 2238 3522 50  0000 L CNN
-F 1 "1kΩ" H 2243 3450 50  0000 L CNN
-F 2 "" V 2240 3440 50  0001 C CNN
-F 3 "~" H 2200 3450 50  0001 C CNN
-	1    2200 3450
-	1    0    0    -1
-$EndComp
-$Comp
-L S2020-rescue:R_US-sDevice Rs
-U 1 1 5F2E19BF
-P 1550 3200
-F 0 "Rs" V 1638 3146 50  0000 L CNN
-F 1 "1kΩ" V 1463 3124 50  0000 L CNN
-F 2 "" V 1590 3190 50  0001 C CNN
-F 3 "~" H 1550 3200 50  0001 C CNN
-	1    1550 3200
-	0    -1   -1   0
-$EndComp
-Wire Wire Line
-	1850 3600 1850 3700
-Wire Wire Line
-	2200 3200 2200 3300
-Wire Wire Line
-	2200 3600 2200 3700
-Text Notes 1824 3176 0    50   ~ 0
-B
-Connection ~ 1850 3200
-Wire Wire Line
-	1850 3200 2200 3200
-Wire Wire Line
-	1850 3200 1850 3300
-Wire Wire Line
-	1700 3200 1850 3200
-$Comp
-L 00TJR:ZENER-RESCUE-F2018 D1
-U 1 1 5F2E19CD
-P 1850 3450
-F 0 "D1" V 1776 3514 50  0000 L CNN
-F 1 "1N4735A" V 1848 3508 30  0000 L CNN
-F 2 "" H 1850 3450 50  0000 C CNN
-F 3 "" H 1850 3450 50  0000 C CNN
-	1    1850 3450
-	0    1    1    0
-$EndComp
-Wire Wire Line
-	1400 3200 1250 3200
-Text Notes 1224 3176 0    50   ~ 0
-A
-$Comp
-L 00TJR:GND #PWR?
-U 1 1 5F2E37ED
-P 1850 3700
-F 0 "#PWR?" H 1850 3450 50  0001 C CNN
-F 1 "GND" H 1900 3500 50  0001 C CNN
-F 2 "" H 1850 3700 50  0000 C CNN
-F 3 "" H 1850 3700 50  0000 C CNN
-	1    1850 3700
-	1    0    0    -1
-$EndComp
-$Comp
-L 00TJR:GND #PWR?
-U 1 1 5F2E3FCC
-P 2200 3700
-F 0 "#PWR?" H 2200 3450 50  0001 C CNN
-F 1 "GND" H 2250 3500 50  0001 C CNN
-F 2 "" H 2200 3700 50  0000 C CNN
-F 3 "" H 2200 3700 50  0000 C CNN
-	1    2200 3700
-	1    0    0    -1
-$EndComp
-$Comp
 L S2020-rescue:CP1-sDevice C?
 U 1 1 5F2E9FE5
@@
 	1    0    0    -1
 $EndComp
-Connection ~ 1250 3200
+$Comp
+L S2020-rescue:R_US-sDevice RL?
+U 1 1 5F3482E7
+P 2750 3300
+F 0 "RL?" H 2788 3372 50  0000 L CNN
+F 1 "1kΩ" H 2793 3300 50  0000 L CNN
+F 2 "" V 2790 3290 50  0001 C CNN
+F 3 "~" H 2750 3300 50  0001 C CNN
+	1    2750 3300
+	1    0    0    -1
+$EndComp
+$Comp
+L S2020-rescue:R_US-sDevice Rs?
+U 1 1 5F3482ED
+P 2000 3000
+F 0 "Rs?" V 2088 2946 50  0000 L CNN
+F 1 "1kΩ 2W" V 1900 2850 50  0000 L CNN
+F 2 "" V 2040 2990 50  0001 C CNN
+F 3 "~" H 2000 3000 50  0001 C CNN
+	1    2000 3000
+	0    -1   -1   0
+$EndComp
+Wire Wire Line
+	2300 3450 2300 3500
+Wire Wire Line
+	2750 3000 2750 3150
+Wire Wire Line
+	2750 3450 2750 3500
+Text Notes 2274 2976 0    50   ~ 0
+B
+Connection ~ 2300 3000
+Wire Wire Line
+	2300 3000 2750 3000
+Wire Wire Line
+	2300 3000 2300 3150
+Wire Wire Line
+	2150 3000 2300 3000
+$Comp
+L 00TJR:ZENER-RESCUE-F2018 D?
+U 1 1 5F3482FB
+P 2300 3300
+F 0 "D?" V 2226 3364 50  0000 L CNN
+F 1 "1N4735A" V 2298 3358 30  0000 L CNN
+F 2 "" H 2300 3300 50  0000 C CNN
+F 3 "" H 2300 3300 50  0000 C CNN
+	1    2300 3300
+	0    1    1    0
+$EndComp
+Text Notes 1674 2976 0    50   ~ 0
+A
+$Comp
+L 00TJR:GND #PWR?
+U 1 1 5F348303
+P 2300 3500
+F 0 "#PWR?" H 2300 3250 50  0001 C CNN
+F 1 "GND" H 2350 3300 50  0001 C CNN
+F 2 "" H 2300 3500 50  0000 C CNN
+F 3 "" H 2300 3500 50  0000 C CNN
+	1    2300 3500
+	1    0    0    -1
+$EndComp
+$Comp
+L 00TJR:GND #PWR?
+U 1 1 5F348309
+P 2750 3500
+F 0 "#PWR?" H 2750 3250 50  0001 C CNN
+F 1 "GND" H 2800 3300 50  0001 C CNN
+F 2 "" H 2750 3500 50  0000 C CNN
+F 3 "" H 2750 3500 50  0000 C CNN
+	1    2750 3500
+	1    0    0    -1
+$EndComp
+Wire Wire Line
+	1850 3000 1700 3000
+Connection ~ 1700 3000
 $EndSCHEMATC
