File: S2020/BJT-Amps.sch (KiCad schematic (older format))
At the start: 35 parts, among them Q1 2N3904

Commit message: mess
Parts:
- removed RE (x2): 820Ω, symbol S2020-rescue:R_US-Device
- added RE10, RE13: 680Ω, symbol S2020-rescue:R_US-Device
- added RE12, RE6, RE9: 150Ω, symbol S2020-rescue:R_US-Device
- C16, C19, C23: renamed from C1; value 10µF -> 1µF
- C17, C20, C22: renamed from C2; value 10µF -> 1µF
- C18, C21: renamed from C3; value 100µF -> 1µF
- R20, R23, R28: renamed from R?; value Rgen -> 50Ω
- RE11, RE14, RE8: renamed from RL; value 680Ω -> 3.3kΩ
- RE7: renamed from RE; value 820Ω -> 680Ω
- gave numbers to parts that had none: 3
- renumbered Q1 to Q10, Q1 to Q11, Q1 to Q12, R1 to R21, R2 to R22, R1 to R24, R2 to R25, R1 to R26, R2 to R27, RC to RC7, RC to RC8, RC to RC9, VCC to VCC07, VCC to VCC08, VCC to VCC09
Connections:
- net GND: now also RE10.2, RE13.2
- net at C18.2, RE7.1: now also RE6.2; no longer Q10.1 (E)
- net at C20.2, Q11.1 (E): now also RE9.1
- net at C23.2: now also RE12.2, RE13.1; no longer Q12.1 (E)
- new net: Q10.1 (E), RE6.1
- new net: Q12.1 (E), RE12.1
- new net: RE10.1, RE9.2
Other:
- note added: "10kHz"
- note added: "20mvp"
- moved on the sheet: C18, C21, C22, C23, R27, RE14, RE7, RE8
