File: S2020/BJT-Bias.sch (KiCad schematic (older format))
At the start: 29 parts, among them Q1 2N3904

Commit message: mess
Parts:
- added Q6: 2N3904, TO-92, symbol 00TJR:2N3904
- added R16: 75kΩ, symbol S2020-rescue:R_US-Device
- added R17: 16kΩ, symbol S2020-rescue:R_US-Device
- added RC3: 2.2kΩ, symbol S2020-rescue:R_US-Device
- added RE2: 680Ω, symbol S2020-rescue:R_US-Device
- added VCC03: +24V, symbol power:+24V
- Q3: renamed from Q?; symbol Transistor_BJT:2N3906 -> S2020-rescue:2N3906-Transistor_BJT
- gave numbers to parts that had none: 2
- renumbered Q1 to Q2, Q1 to Q5, Q1 to Q7, Q1 to Q8, Q1 to Q9, R1 to R18, R2 to R19, RB to RB1, RB to RB2, RB to RB3, RB to RB4, RC to RC1, RC to RC2, RC to RC4, RC to RC5, RC to RC6, RE to RE1, RE to RE3, RE to RE4, RE to RE5, VCC to VCC01, VCC to VCC02, VCC to VCC04, VCC to VCC05, VCC to VCC6, VEE to VEE1
Connections:
- net +24V: now also R16.1, RC3.1, VCC03.1 (+24V)
- net GND: now also R17.2, RE2.2
- new net: Q6.~ (E), RC3.2
- new net: Q6.~ (E), R16.2, R17.1
- new net: Q6.~ (E), RE2.1
