File: S2020/Clampers.sch (KiCad schematic (older format))
At the start: 8 parts

Commit message: mess
Parts:
- renumbered 2vp to 2vp1, 2vp to 2vp2, C1 to C5, C1 to C6, D1 to D10, D1 to D11, R1 to R14, R1 to R15
Changed lines of the file:
@@
 EESchema Schematic File Version 4
+LIBS:S2020-cache
 EELAYER 30 0
 EELAYER END
 $Descr A 11000 8500
 encoding utf-8
-Sheet 4 13
+Sheet 4 14
 Title "Clampers"
 Date ""
@@
 $EndDescr
 $Comp
-L 00TJR:C C1
+L 00TJR:C C5
 U 1 1 5E22F73C
 P 1900 1300
-F 0 "C1" V 1756 1300 50  0000 C CNN
+F 0 "C5" V 1756 1300 50  0000 C CNN
 F 1 "1µF" V 2036 1300 50  0000 C CNN
 F 2 "" H 1938 1150 50  0000 C CNN
@@
 $EndComp
 $Comp
-L Device:R_US R1
+L Device:R_US R14
 U 1 1 5E22FC20
 P 2750 1650
-F 0 "R1" H 2796 1713 50  0000 L CNN
+F 0 "R14" H 2796 1713 50  0000 L CNN
 F 1 "10kΩ" H 2797 1636 50  0000 L CNN
 F 2 "" V 2790 1640 50  0001 C CNN
@@
 $EndComp
 $Comp
-L 00TJR:D D1
+L 00TJR:D D10
 U 1 1 5E230A0F
 P 2300 1650
-F 0 "D1" V 2322 1598 50  0000 R CNN
+F 0 "D10" V 2322 1598 50  0000 R CNN
 F 1 "D" V 2255 1572 50  0001 R CNN
 F 2 "" H 2300 1650 50  0000 C CNN
@@
 $EndComp
 $Comp
-L 00TJR:Vgen 2vp
+L 00TJR:Vgen 2vp1
 U 1 1 5E231506
 P 1500 1650
-F 0 "2vp" H 1314 1773 50  0000 L CNN
+F 0 "2vp1" H 1314 1773 50  0000 L CNN
 F 1 "1kHz" H 1307 1513 50  0000 L CNN
 F 2 "" V 1500 1690 50  0000 C CNN
@@
 	2300 2000 1500 2000
 $Comp
-L 00TJR:GND #PWR?
+L 00TJR:GND #PWR022
 U 1 1 5E237C5D
 P 1500 2050
-F 0 "#PWR?" H 1500 1800 50  0001 C CNN
+F 0 "#PWR022" H 1500 1800 50  0001 C CNN
 F 1 "GND" H 1505 1877 50  0001 C CNN
 F 2 "" H 1500 2050 50  0000 C CNN
@@
 B
 $Comp
-L 00TJR:C C1
+L 00TJR:C C6
 U 1 1 5E23B8A3
 P 4100 1300
-F 0 "C1" V 3956 1300 50  0000 C CNN
+F 0 "C6" V 3956 1300 50  0000 C CNN
 F 1 "1µF" V 4236 1300 50  0000 C CNN
 F 2 "" H 4138 1150 50  0000 C CNN
@@
 $EndComp
 $Comp
-L Device:R_US R1
+L Device:R_US R15
 U 1 1 5E23B8A9
 P 4950 1650
-F 0 "R1" H 4996 1713 50  0000 L CNN
+F 0 "R15" H 4996 1713 50  0000 L CNN
 F 1 "10kΩ" H 4997 1636 50  0000 L CNN
 F 2 "" V 4990 1640 50  0001 C CNN
@@
 $EndComp
 $Comp
-L 00TJR:Vgen 2vp
+L 00TJR:Vgen 2vp2
 U 1 1 5E23B8B5
 P 3700 1650
-F 0 "2vp" H 3514 1773 50  0000 L CNN
+F 0 "2vp2" H 3514 1773 50  0000 L CNN
 F 1 "1kHz" H 3507 1513 50  0000 L CNN
 F 2 "" V 3700 1690 50  0000 C CNN
@@
 	4500 2000 3700 2000
 $Comp
-L 00TJR:GND #PWR?
+L 00TJR:GND #PWR023
 U 1 1 5E23B8C8
 P 3700 2050
-F 0 "#PWR?" H 3700 1800 50  0001 C CNN
+F 0 "#PWR023" H 3700 1800 50  0001 C CNN
 F 1 "GND" H 3705 1877 50  0001 C CNN
 F 2 "" H 3700 2050 50  0000 C CNN
@@
 B
 $Comp
-L 00TJR:D D1
+L 00TJR:D D11
 U 1 1 5E23B8AF
 P 4500 1650
-F 0 "D1" V 4522 1598 50  0000 R CNN
+F 0 "D11" V 4522 1598 50  0000 R CNN
 F 1 "D" V 4455 1572 50  0001 R CNN
 F 2 "" H 4500 1650 50  0000 C CNN
