File: S2020/Clipper.sch (KiCad schematic (older format))
At the start: 6 parts

Commit message: mess
Parts:
- renumbered 1kHz to 1kHz1, 1kHz to 1kHz2, D1 to D8, D1 to D9, R1 to R12, R1 to R13
Changed lines of the file:
@@
 EESchema Schematic File Version 4
+LIBS:S2020-cache
 EELAYER 30 0
 EELAYER END
 $Descr USLetter 11000 8500
 encoding utf-8
-Sheet 3 13
+Sheet 3 14
 Title "Clipper"
 Date "2020-01-07"
@@
 $EndDescr
 $Comp
-L 00TJR:Vgen 1kHz
+L 00TJR:Vgen 1kHz1
 U 1 1 5E14BA44
 P 1000 1300
-F 0 "1kHz" H 802 1161 50  0000 L CNN
+F 0 "1kHz1" H 802 1161 50  0000 L CNN
 F 1 "10vp" H 807 1450 50  0000 L CNN
 F 2 "" V 1000 1340 50  0000 C CNN
@@
 $EndComp
 $Comp
-L S2020-rescue:D_ALT-sDevice D1
+L S2020-rescue:D_ALT-sDevice D8
 U 1 1 5E14E31A
 P 1400 950
-F 0 "D1" H 1403 1047 50  0000 C CNN
+F 0 "D8" H 1403 1047 50  0000 C CNN
 F 1 "1N4001" H 1412 858 50  0000 C CNN
 F 2 "" H 1400 950 50  0001 C CNN
@@
 $EndComp
 $Comp
-L 00TJR:GND #PWR01
+L 00TJR:GND #PWR020
 U 1 1 5E14EB0D
 P 1000 1700
-F 0 "#PWR01" H 1000 1450 50  0001 C CNN
+F 0 "#PWR020" H 1000 1450 50  0001 C CNN
 F 1 "GND" H 1050 1500 50  0001 C CNN
 F 2 "" H 1000 1700 50  0000 C CNN
@@
 Connection ~ 1000 1650
 $Comp
-L S2020-rescue:R_US-sDevice R1
+L S2020-rescue:R_US-sDevice R12
 U 1 1 5E14E4A3
 P 1750 1300
-F 0 "R1" H 1792 1402 50  0000 L CNN
+F 0 "R12" H 1792 1402 50  0000 L CNN
 F 1 "10kΩ" H 1792 1329 50  0000 L CNN
 F 2 "" V 1790 1290 50  0001 C CNN
@@
 	1000 1650 1000 1700
 $Comp
-L S2020-rescue:D_ALT-sDevice D1
+L S2020-rescue:D_ALT-sDevice D9
 U 1 1 5E15DF7B
 P 2900 950
-F 0 "D1" H 2903 1047 50  0000 C CNN
+F 0 "D9" H 2903 1047 50  0000 C CNN
 F 1 "1N4001" H 2912 858 50  0000 C CNN
 F 2 "" H 2900 950 50  0001 C CNN
@@
 $EndComp
 $Comp
-L 00TJR:GND #PWR02
+L 00TJR:GND #PWR021
 U 1 1 5E15DF81
 P 2500 1700
-F 0 "#PWR02" H 2500 1450 50  0001 C CNN
+F 0 "#PWR021" H 2500 1450 50  0001 C CNN
 F 1 "GND" H 2550 1500 50  0001 C CNN
 F 2 "" H 2500 1700 50  0000 C CNN
@@
 Connection ~ 2500 1650
 $Comp
-L S2020-rescue:R_US-sDevice R1
+L S2020-rescue:R_US-sDevice R13
 U 1 1 5E15DF8F
 P 3250 1300
-F 0 "R1" H 3292 1402 50  0000 L CNN
+F 0 "R13" H 3292 1402 50  0000 L CNN
 F 1 "10kΩ" H 3292 1329 50  0000 L CNN
 F 2 "" V 3290 1290 50  0001 C CNN
@@
 	2500 1650 2500 1700
 $Comp
-L 00TJR:Vgen 1kHz
+L 00TJR:Vgen 1kHz2
 U 1 1 5E15ECD9
 P 2500 1300
-F 0 "1kHz" H 2302 1161 50  0000 L CNN
+F 0 "1kHz2" H 2302 1161 50  0000 L CNN
 F 1 "10vp" H 2307 1450 50  0000 L CNN
 F 2 "" V 2500 1340 50  0000 C CNN
