File: S2020/FET.sch (KiCad schematic (older format))
At the start: 43 parts, among them Q1 2N5951, Q1 BS170

Commit message: mess
Parts:
- removed +18V: VDD, symbol power:VDD
- removed 10kHz: 250mvp, symbol 00TJR:Vgen
- removed C1: 10µF, symbol Device:C
- removed Q1 (x4): 2N5951, symbol Device:Q_NJFET_GSD
- removed Q1 (x2): BS170, Package_TO_SOT_THT:TO-92_Inline, symbol Transistor_FET:BS170
- removed R?: Rgen, symbol 00TJR:Rgen
- removed RD: 1kΩ, symbol S2020-rescue:R_US-Device
- removed VGS (x2): 0-5V, symbol 00TJR:Battery
- added +15V02: VDD, symbol power:VDD
- added 10kHz1: 250mvp, symbol 00TJR:Vgen
- added C27: 1µF, symbol Device:C
- added Q13, Q15, Q17, Q20: 2N5951, symbol 00TJR:NJFET
- added Q14, Q16: BS170, Package_TO_SOT_THT:TO-92_Inline, symbol 00TJR:NEMOSFET
- added Q18: N-Channel, symbol 00TJR:NJFET
- added Q21: P-Channel, symbol 00TJR:PJFET
- added R32: 50Ω, symbol 00TJR:Rgen
- added RC11: 1kΩ, symbol S2020-rescue:R_US-Device
- added VGS1, VGS2: 0V to 5V, symbol 00TJR:VarDC
- added Vm1, Vm2, Vm3: 1V=1mA, symbol 00TJR:VoltMeter
- C24: renamed from C1; value 10µF -> 1µF
- C25, C28: renamed from C2; value 10µF -> 1µF
- C26, C29: renamed from C3; value 100µF -> 1µF
- R29: renamed from R?; value Rgen -> 50Ω
- RE16, RL3: renamed from RL; value 10kΩ -> 4.7kΩ
- RG1: renamed from RG; value 120kΩ -> 22kΩ
- gave numbers to parts that had none: 4
- renumbered +18V to +15V01, +18V to +15V03, +18V to +15V04, +18V to +15V05, +18V to +15V06, 10kHz to G5, R2 to R30, RG to R31, RD to RC10, RD to RC12, RD to RC13, RD to RD1, RD to RD2, RS to RE15, RG to RG2, RS to RS1, RS to RS2
Connections:
- net GND: now also 10kHz1.2, Q13.1 (G), Q13.2 (S), Q14.3 (S), Q15.2 (S), VGS1.2, VGS2.1
- net VDD: now also +15V02.1 (VDD), RC11.1
- net at RC13.2: now also Q17.3 (D)
- net at RE15.1: now also Q17.2 (S)
- net at R31.1: now also Q17.1 (G)
- net at C28.2, RD2.2: now also Q20.3 (D)
- net at C24.1: now also R30.1, RG1.2, Q16.2 (G); no longer RG2.1
- net at C29.2, RS2.1: now also Q20.2 (S)
- net at RC12.2: now also Q15.3 (D)
- net at RC10.2: now also Q13.3 (D)
- net at C25.2, RD1.2: now also Q16.1 (D)
- net at C26.2, RS1.1: now also Q16.3 (S)
- new net: C27.1, Q20.1 (G), RG2.1
- new net: Q15.1 (G), VGS2.2
- new net: 10kHz1.1, R32.2
- new net: C27.2, R32.1
- new net: Q14.1 (D), RC11.2
- new net: Q14.2 (G), VGS1.1
Other:
- moved on the sheet: C24, C28, C29, MES1, R31, RC10, RC12, RC13, RD2, RE15, RE16, RG2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
