File: S2020/S2020.sch (KiCad schematic (older format))
At the start: 13 parts

Commit message: mess
Parts:
- gave numbers to parts that had none: 13
Changed lines of the file:
@@
 EESchema Schematic File Version 4
+LIBS:S2020-cache
 EELAYER 30 0
 EELAYER END
 $Descr USLetter 11000 8500
 encoding utf-8
-Sheet 1 13
+Sheet 1 14
 Title "AC/DC"
 Date "2020-01-06"
@@
 $EndDescr
 $Comp
-L S2020-rescue:R_US-Device R?
+L S2020-rescue:R_US-Device R2
 U 1 1 5E04B9A2
 P 2700 1350
-F 0 "R?" H 2748 1429 50  0000 L CNN
+F 0 "R2" H 2748 1429 50  0000 L CNN
 F 1 "20kΩ" H 2745 1357 50  0000 L CNN
 F 2 "" V 2740 1340 50  0001 C CNN
@@
 $EndComp
 $Comp
-L S2020-rescue:GND-power #PWR?
+L S2020-rescue:GND-power #PWR03
 U 1 1 5E04CFCE
 P 2700 2400
-F 0 "#PWR?" H 2700 2150 50  0001 C CNN
+F 0 "#PWR03" H 2700 2150 50  0001 C CNN
 F 1 "GND" H 2705 2227 50  0001 C CNN
 F 2 "" H 2700 2400 50  0001 C CNN
@@
 $EndComp
 $Comp
-L S2020-rescue:C_Small-Device C?
+L S2020-rescue:C_Small-Device C2
 U 1 1 5E04EB10
 P 3150 2100
-F 0 "C?" H 3216 2175 50  0000 L CNN
+F 0 "C2" H 3216 2175 50  0000 L CNN
 F 1 "100pF" H 3224 2100 50  0000 L CNN
 F 2 "" H 3150 2100 50  0001 C CNN
@@
 $EndComp
 $Comp
-L S2020-rescue:R_US-Device R?
+L S2020-rescue:R_US-Device R3
 U 1 1 5E04E37A
 P 2700 2100
-F 0 "R?" H 2748 2175 50  0000 L CNN
+F 0 "R3" H 2748 2175 50  0000 L CNN
 F 1 "3.3kΩ" H 2754 2100 50  0000 L CNN
 F 2 "" V 2740 2090 50  0001 C CNN
@@
 	3150 2200 3150 2400
 $Comp
-L S2020-rescue:GND-power #PWR?
+L S2020-rescue:GND-power #PWR04
 U 1 1 5E05590C
 P 3150 2400
-F 0 "#PWR?" H 3150 2150 50  0001 C CNN
+F 0 "#PWR04" H 3150 2150 50  0001 C CNN
 F 1 "GND" H 3155 2227 50  0001 C CNN
 F 2 "" H 3150 2400 50  0001 C CNN
@@
 Connection ~ 3150 1700
 $Comp
-L S2020-rescue:TestPoint-Connector TP?
+L S2020-rescue:TestPoint-Connector TP2
 U 1 1 5E0639ED
 P 3150 1700
-F 0 "TP?" H 3092 1897 50  0000 L CNN
+F 0 "TP2" H 3092 1897 50  0000 L CNN
 F 1 "TestPoint" H 3208 1727 50  0001 L CNN
 F 2 "" H 3350 1700 50  0001 C CNN
@@
 Connection ~ 1200 1700
 $Comp
-L S2020-rescue:TestPoint-Connector TP?
+L S2020-rescue:TestPoint-Connector TP1
 U 1 1 5E063233
 P 1200 1700
-F 0 "TP?" H 1137 1897 50  0000 L CNN
+F 0 "TP1" H 1137 1897 50  0000 L CNN
 F 1 "TestPoint" H 1258 1727 50  0001 L CNN
 F 2 "" H 1400 1700 50  0001 C CNN
@@
 	1200 1700 1200 1800
 $Comp
-L 00TJR:Rgen Rgen?
+L 00TJR:Rgen Rgen1
 U 1 1 5E057D02
 P 1200 1900
-F 0 "Rgen?" H 997 1961 50  0000 L CNN
+F 0 "Rgen1" H 997 1961 50  0000 L CNN
 F 1 "50Ω" H 1003 1881 50  0000 L CNN
 F 2 "" V 1130 1900 50  0000 C CNN
@@
 $EndComp
 $Comp
-L S2020-rescue:GND-power #PWR?
+L S2020-rescue:GND-power #PWR01
 U 1 1 5E055587
 P 1200 2400
-F 0 "#PWR?" H 1200 2150 50  0001 C CNN
+F 0 "#PWR01" H 1200 2150 50  0001 C CNN
 F 1 "GND" H 1205 2227 50  0001 C CNN
 F 2 "" H 1200 2400 50  0001 C CNN
@@
 $EndComp
 $Comp
-L S2020-rescue:C_Small-Device C?
+L S2020-rescue:C_Small-Device C1
 U 1 1 5E04BE92
 P 1650 1700
-F 0 "C?" V 1528 1660 50  0000 L CNN
+F 0 "C1" V 1528 1660 50  0000 L CNN
 F 1 "0.1µF" V 1754 1597 50  0000 L CNN
 F 2 "" H 1650 1700 50  0001 C CNN
@@
 $EndComp
 $Comp
-L 00TJR:Vgen G?
+L 00TJR:Vgen G1
 U 1 1 5E0504F3
 P 1200 2200
-F 0 "G?" H 900 2250 50  0001 L CNN
+F 0 "G1" H 900 2250 50  0001 L CNN
 F 1 "4vp" H 994 2292 50  0000 L CNN
 F 2 "" V 1200 2240 50  0000 C CNN
@@
 $EndComp
 $Comp
-L S2020-rescue:R_US-Device R?
+L S2020-rescue:R_US-Device R1
 U 1 1 5E066804
 P 2200 1700
-F 0 "R?" V 2109 1649 50  0000 L CNN
+F 0 "R1" V 2109 1649 50  0000 L CNN
 F 1 "2kΩ" V 2281 1623 50  0000 L CNN
 F 2 "" V 2240 1690 50  0001 C CNN
@@
 	1750 1700 2050 1700
 $Comp
-L S2020-rescue:+10V-power #PWR?
+L S2020-rescue:+10V-power #PWR02
 U 1 1 5E0773F2
 P 2700 1100
-F 0 "#PWR?" H 2700 950 50  0001 C CNN
+F 0 "#PWR02" H 2700 950 50  0001 C CNN
 F 1 "+10V" H 2715 1273 50  0000 C CNN
 F 2 "" H 2700 1100 50  0001 C CNN
@@
 $EndSheet
 $Comp
-L S2020-rescue:R_US-Device R?
+L S2020-rescue:R_US-Device R6
 U 1 1 5E4859CC
 P 16400 3400
-F 0 "R?" H 16448 3475 50  0001 L CNN
+F 0 "R6" H 16448 3475 50  0001 L CNN
 F 1 "3.3kΩ" H 16454 3400 50  0001 L CNN
 F 2 "" V 16440 3390 50  0001 C CNN
@@
 $EndComp
 $Comp
-L S2020-rescue:GND-power #PWR?
+L S2020-rescue:GND-power #PWR07
 U 1 1 5E485DF9
 P 16400 3550
-F 0 "#PWR?" H 16400 3300 50  0001 C CNN
+F 0 "#PWR07" H 16400 3300 50  0001 C CNN
 F 1 "GND" H 16405 3377 50  0001 C CNN
 F 2 "" H 16400 3550 50  0001 C CNN
@@
 	16400 3250 16400 3150
 $Comp
-L S2020-rescue:R_US-Device R?
+L S2020-rescue:R_US-Device R5
 U 1 1 5E4FCABC
 P 15600 3400
-F 0 "R?" H 15648 3475 50  0001 L CNN
+F 0 "R5" H 15648 3475 50  0001 L CNN
 F 1 "3.3kΩ" H 15654 3400 50  0001 L CNN
 F 2 "" V 15640 3390 50  0001 C CNN
@@
 $EndComp
 $Comp
-L S2020-rescue:GND-power #PWR?
+L S2020-rescue:GND-power #PWR06
 U 1 1 5E4FD25A
 P 15600 3550
-F 0 "#PWR?" H 15600 3300 50  0001 C CNN
+F 0 "#PWR06" H 15600 3300 50  0001 C CNN
 F 1 "GND" H 15605 3377 50  0001 C CNN
 F 2 "" H 15600 3550 50  0001 C CNN
@@
 	15600 3150 14300 3150
 $Comp
-L S2020-rescue:R_US-Device R?
+L S2020-rescue:R_US-Device R4
 U 1 1 5E5041BE
 P 14300 3400
-F 0 "R?" H 14348 3475 50  0001 L CNN
+F 0 "R4" H 14348 3475 50  0001 L CNN
 F 1 "3.3kΩ" H 14354 3400 50  0001 L CNN
 F 2 "" V 14340 3390 50  0001 C CNN
@@
 $EndComp
 $Comp
-L S2020-rescue:R_US-Device R?
+L S2020-rescue:R_US-Device R7
 U 1 1 5E504699
 P 17900 3400
-F 0 "R?" H 17948 3475 50  0001 L CNN
+F 0 "R7" H 17948 3475 50  0001 L CNN
 F 1 "3.3kΩ" H 17954 3400 50  0001 L CNN
 F 2 "" V 17940 3390 50  0001 C CNN
@@
 $EndComp
 $Comp
-L S2020-rescue:GND-power #PWR?
+L S2020-rescue:GND-power #PWR05
 U 1 1 5E50534C
 P 14300 3550
-F 0 "#PWR?" H 14300 3300 50  0001 C CNN
+F 0 "#PWR05" H 14300 3300 50  0001 C CNN
 F 1 "GND" H 14305 3377 50  0001 C CNN
 F 2 "" H 14300 3550 50  0001 C CNN
@@
 $EndComp
 $Comp
-L S2020-rescue:GND-power #PWR?
+L S2020-rescue:GND-power #PWR08
 U 1 1 5E5056E0
 P 17900 3550
-F 0 "#PWR?" H 17900 3300 50  0001 C CNN
+F 0 "#PWR08" H 17900 3300 50  0001 C CNN
 F 1 "GND" H 17905 3377 50  0001 C CNN
 F 2 "" H 17900 3550 50  0001 C CNN
@@
 F1 "temp.sch" 50
 $EndSheet
+$Sheet
+S 11100 11150 2550 1450
+U 5F5FC6BE
+F0 "Multistage" 50
+F1 "Multistage.sch" 50
+$EndSheet
 $EndSCHEMATC
