File: S2020/Switching.sch (KiCad schematic (older format))
At the start: 72 parts, among them Q1 2N3904, Q2 2N3904, SW1 SW_Push, SW2 SW_Push, SW3 SW_Push, U1 LM741

Commit message: mess
Parts:
- gave numbers to parts that had none: 26
- renumbered D1 to D23, D1 to D24, D1 to D25, D1 to D26, D1 to D27, D1 to D28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
