File: S2020/Voltage Multipliers.sch (KiCad schematic (older format))
At the start: 32 parts, among them T1 4:1

Commit message: mess
Parts:
- renumbered 40vp to 40vp1, 40vp to 40vp2, 40vp to 40vp3, C2 to C10, C1 to C11, C3 to C12, C2 to C13, C4 to C14, C3 to C15, C1 to C7, C1 to C8, C2 to C9, D1 to D12, D1 to D13, D2 to D14, D2 to D15, D1 to D16, D3 to D17, D2 to D18, D4 to D19, D3 to D20, T1 to T3, T1 to T4, T1 to T5, D to TP10, A to TP3, F to TP4, B to TP5, TP1 to TP6, TP2 to TP7, E to TP8, C to TP9
Changed lines of the file:
@@
 EESchema Schematic File Version 4
+LIBS:S2020-cache
 EELAYER 30 0
 EELAYER END
 $Descr A 11000 8500
 encoding utf-8
-Sheet 5 13
+Sheet 5 14
 Title ""
 Date ""
@@
 P 2450 1600
 AR Path="/5E22ED3E/5E23E293" Ref="D?"  Part="1"
-AR Path="/5E23D312/5E23E293" Ref="D1"  Part="1"
-F 0 "D1" H 2502 1509 50  0000 R CNN
+AR Path="/5E23D312/5E23E293" Ref="D13"  Part="1"
+F 0 "D13" H 2502 1509 50  0000 R CNN
 F 1 "D" V 2405 1522 50  0001 R CNN
 F 2 "" H 2450 1600 50  0000 C CNN
@@
 $EndComp
 $Comp
-L 00TJR:TRANSFOIron T1
+L 00TJR:TRANSFOIron T4
 U 1 1 5E23EEE0
 P 1600 1800
-F 0 "T1" H 1601 2058 50  0000 C CNN
+F 0 "T4" H 1601 2058 50  0000 C CNN
 F 1 "4:1" H 1598 1547 50  0000 C CNN
 F 2 "" H 1600 1800 50  0000 C CNN
@@
 P 2450 2400
 AR Path="/5E22ED3E/5E23F8F7" Ref="D?"  Part="1"
-AR Path="/5E23D312/5E23F8F7" Ref="D2"  Part="1"
-F 0 "D2" H 2500 2300 50  0000 R CNN
+AR Path="/5E23D312/5E23F8F7" Ref="D14"  Part="1"
+F 0 "D14" H 2500 2300 50  0000 R CNN
 F 1 "D" V 2405 2322 50  0001 R CNN
 F 2 "" H 2450 2400 50  0000 C CNN
@@
 $EndComp
 $Comp
-L 00TJR:CP1_Small C1
+L 00TJR:CP1_Small C8
 U 1 1 5E23FFA8
 P 2700 1800
-F 0 "C1" H 2791 1846 50  0000 L CNN
+F 0 "C8" H 2791 1846 50  0000 L CNN
 F 1 "10µF" H 2791 1755 50  0000 L CNN
 F 2 "" H 2700 1800 50  0000 C CNN
@@
 $EndComp
 $Comp
-L 00TJR:CP1_Small C2
+L 00TJR:CP1_Small C9
 U 1 1 5E240374
 P 2700 2200
-F 0 "C2" H 2791 2246 50  0000 L CNN
+F 0 "C9" H 2791 2246 50  0000 L CNN
 F 1 "10µF" H 2791 2155 50  0000 L CNN
 F 2 "" H 2700 2200 50  0000 C CNN
@@
 P 3000 1600
 AR Path="/5E24753A" Ref="TP?"  Part="1"
-AR Path="/5E23D312/5E24753A" Ref="TP1"  Part="1"
-F 0 "TP1" V 2917 1668 50  0000 L CNN
+AR Path="/5E23D312/5E24753A" Ref="TP6"  Part="1"
+F 0 "TP6" V 2917 1668 50  0000 L CNN
 F 1 "TestPoint" H 3058 1627 50  0001 L CNN
 F 2 "" H 3200 1600 50  0001 C CNN
@@
 P 3000 2400
 AR Path="/5E2478E1" Ref="TP?"  Part="1"
-AR Path="/5E23D312/5E2478E1" Ref="TP2"  Part="1"
-F 0 "TP2" V 2921 2473 50  0000 L CNN
+AR Path="/5E23D312/5E2478E1" Ref="TP7"  Part="1"
+F 0 "TP7" V 2921 2473 50  0000 L CNN
 F 1 "TestPoint" H 3058 2427 50  0001 L CNN
 F 2 "" H 3200 2400 50  0001 C CNN
@@
 $EndComp
 $Comp
-L 00TJR:Vgen 40vp
+L 00TJR:Vgen 40vp1
 U 1 1 5E247FD8
 P 1100 1800
-F 0 "40vp" H 905 1949 50  0000 L CNN
+F 0 "40vp1" H 905 1949 50  0000 L CNN
 F 1 "60Hz" H 900 1666 50  0000 L CNN
 F 2 "" V 1100 1840 50  0000 C CNN
@@
 	1200 2000 1100 2000
 $Comp
-L 00TJR:Vgen 40vp
+L 00TJR:Vgen 40vp3
 U 1 1 5E24A4D0
 P 1800 3750
-F 0 "40vp" H 1605 3899 50  0000 L CNN
+F 0 "40vp3" H 1605 3899 50  0000 L CNN
 F 1 "60Hz" H 1600 3616 50  0000 L CNN
 F 2 "" V 1800 3790 50  0000 C CNN
@@
 $EndComp
 $Comp
-L 00TJR:TRANSFOIron T1
+L 00TJR:TRANSFOIron T5
 U 1 1 5E24A9FE
 P 2250 3750
-F 0 "T1" H 2251 4008 50  0000 C CNN
+F 0 "T5" H 2251 4008 50  0000 C CNN
 F 1 "4:1" H 2248 3497 50  0000 C CNN
 F 2 "" H 2250 3750 50  0000 C CNN
@@
 P 3100 3750
 AR Path="/5E22ED3E/5E24C9A1" Ref="D?"  Part="1"
-AR Path="/5E23D312/5E24C9A1" Ref="D1"  Part="1"
-F 0 "D1" V 3146 3695 50  0000 R CNN
+AR Path="/5E23D312/5E24C9A1" Ref="D16"  Part="1"
+F 0 "D16" V 3146 3695 50  0000 R CNN
 F 1 "D" V 3055 3672 50  0001 R CNN
 F 2 "" H 3100 3750 50  0000 C CNN
@@
 $EndComp
 $Comp
-L 00TJR:CP1_Small C2
+L 00TJR:CP1_Small C13
 U 1 1 5E24F7EC
 P 3400 3950
-F 0 "C2" V 3500 3946 50  0000 C CNN
+F 0 "C13" V 3500 3946 50  0000 C CNN
 F 1 "10µF" V 3285 3949 50  0000 C CNN
 F 2 "" H 3400 3950 50  0000 C CNN
@@
 P 3700 3750
 AR Path="/5E22ED3E/5E250CFC" Ref="D?"  Part="1"
-AR Path="/5E23D312/5E250CFC" Ref="D2"  Part="1"
-F 0 "D2" V 3750 3900 50  0000 R CNN
+AR Path="/5E23D312/5E250CFC" Ref="D18"  Part="1"
+F 0 "D18" V 3750 3900 50  0000 R CNN
 F 1 "D" V 3655 3672 50  0001 R CNN
 F 2 "" H 3700 3750 50  0000 C CNN
@@
 $EndComp
 $Comp
-L 00TJR:CP1_Small C3
+L 00TJR:CP1_Small C15
 U 1 1 5E251969
 P 4000 3550
-F 0 "C3" V 4100 3546 50  0000 C CNN
+F 0 "C15" V 4100 3546 50  0000 C CNN
 F 1 "10µF" V 3885 3549 50  0000 C CNN
 F 2 "" H 4000 3550 50  0000 C CNN
@@
 P 4300 3750
 AR Path="/5E22ED3E/5E2526B2" Ref="D?"  Part="1"
-AR Path="/5E23D312/5E2526B2" Ref="D3"  Part="1"
-F 0 "D3" V 4346 3695 50  0000 R CNN
+AR Path="/5E23D312/5E2526B2" Ref="D20"  Part="1"
+F 0 "D20" V 4346 3695 50  0000 R CNN
 F 1 "D" V 4255 3672 50  0001 R CNN
 F 2 "" H 4300 3750 50  0000 C CNN
@@
 Connection ~ 3100 3550
 $Comp
-L 00TJR:CP1_Small C1
+L 00TJR:CP1_Small C11
 U 1 1 5E256ECB
 P 2800 3550
-F 0 "C1" V 2900 3546 50  0000 C CNN
+F 0 "C11" V 2900 3546 50  0000 C CNN
 F 1 "10µF" V 2685 3549 50  0000 C CNN
 F 2 "" H 2800 3550 50  0000 C CNN
@@
 D
 $Comp
-L 00TJR:Vgen 40vp
+L 00TJR:Vgen 40vp2
 U 1 1 5E264454
 P 1100 4750
-F 0 "40vp" H 905 4899 50  0000 L CNN
+F 0 "40vp2" H 905 4899 50  0000 L CNN
 F 1 "60Hz" H 900 4616 50  0000 L CNN
 F 2 "" V 1100 4790 50  0000 C CNN
@@
 $EndComp
 $Comp
-L 00TJR:TRANSFOIron T1
+L 00TJR:TRANSFOIron T3
 U 1 1 5E26445A
 P 1550 4750
-F 0 "T1" H 1551 5008 50  0000 C CNN
+F 0 "T3" H 1551 5008 50  0000 C CNN
 F 1 "4:1" H 1548 4497 50  0000 C CNN
 F 2 "" H 1550 4750 50  0000 C CNN
@@
 P 2400 4750
 AR Path="/5E22ED3E/5E264460" Ref="D?"  Part="1"
-AR Path="/5E23D312/5E264460" Ref="D1"  Part="1"
-F 0 "D1" V 2446 4695 50  0000 R CNN
+AR Path="/5E23D312/5E264460" Ref="D12"  Part="1"
+F 0 "D12" V 2446 4695 50  0000 R CNN
 F 1 "D" V 2355 4672 50  0001 R CNN
 F 2 "" H 2400 4750 50  0000 C CNN
@@
 $EndComp
 $Comp
-L 00TJR:CP1_Small C2
+L 00TJR:CP1_Small C10
 U 1 1 5E264466
 P 2700 4950
-F 0 "C2" V 2800 4946 50  0000 C CNN
+F 0 "C10" V 2800 4946 50  0000 C CNN
 F 1 "10µF" V 2585 4949 50  0000 C CNN
 F 2 "" H 2700 4950 50  0000 C CNN
@@
 P 3000 4750
 AR Path="/5E22ED3E/5E26446C" Ref="D?"  Part="1"
-AR Path="/5E23D312/5E26446C" Ref="D2"  Part="1"
-F 0 "D2" V 3050 4900 50  0000 R CNN
+AR Path="/5E23D312/5E26446C" Ref="D15"  Part="1"
+F 0 "D15" V 3050 4900 50  0000 R CNN
 F 1 "D" V 2955 4672 50  0001 R CNN
 F 2 "" H 3000 4750 50  0000 C CNN
@@
 $EndComp
 $Comp
-L 00TJR:CP1_Small C3
+L 00TJR:CP1_Small C12
 U 1 1 5E264472
 P 3300 4550
-F 0 "C3" V 3400 4546 50  0000 C CNN
+F 0 "C12" V 3400 4546 50  0000 C CNN
 F 1 "10µF" V 3185 4549 50  0000 C CNN
 F 2 "" H 3300 4550 50  0000 C CNN
@@
 P 3600 4750
 AR Path="/5E22ED3E/5E264478" Ref="D?"  Part="1"
-AR Path="/5E23D312/5E264478" Ref="D3"  Part="1"
-F 0 "D3" V 3646 4695 50  0000 R CNN
+AR Path="/5E23D312/5E264478" Ref="D17"  Part="1"
+F 0 "D17" V 3646 4695 50  0000 R CNN
 F 1 "D" V 3555 4672 50  0001 R CNN
 F 2 "" H 3600 4750 50  0000 C CNN
@@
 Connection ~ 2400 4550
 $Comp
-L 00TJR:CP1_Small C1
+L 00TJR:CP1_Small C7
 U 1 1 5E26448F
 P 2100 4550
-F 0 "C1" V 2200 4546 50  0000 C CNN
+F 0 "C7" V 2200 4546 50  0000 C CNN
 F 1 "10µF" V 1985 4549 50  0000 C CNN
 F 2 "" H 2100 4550 50  0000 C CNN
@@
 	1150 4950 1100 4950
 $Comp
-L 00TJR:CP1_Small C4
+L 00TJR:CP1_Small C14
 U 1 1 5E26681A
 P 3900 4950
-F 0 "C4" V 4000 4946 50  0000 C CNN
+F 0 "C14" V 4000 4946 50  0000 C CNN
 F 1 "10µF" V 3785 4949 50  0000 C CNN
 F 2 "" H 3900 4950 50  0000 C CNN
@@
 P 4200 4750
 AR Path="/5E22ED3E/5E266820" Ref="D?"  Part="1"
-AR Path="/5E23D312/5E266820" Ref="D4"  Part="1"
-F 0 "D4" V 4250 4900 50  0000 R CNN
+AR Path="/5E23D312/5E266820" Ref="D19"  Part="1"
+F 0 "D19" V 4250 4900 50  0000 R CNN
 F 1 "D" V 4155 4672 50  0001 R CNN
 F 2 "" H 4200 4750 50  0000 C CNN
@@
 P 1950 4550
 AR Path="/5E24760C" Ref="TP?"  Part="1"
-AR Path="/5E23D312/5E24760C" Ref="A"  Part="1"
-F 0 "A" H 1924 4757 50  0000 L CNN
+AR Path="/5E23D312/5E24760C" Ref="TP3"  Part="1"
+F 0 "TP3" H 1924 4757 50  0000 L CNN
 F 1 "TestPoint" H 2008 4577 50  0001 L CNN
 F 2 "" H 2150 4550 50  0001 C CNN
@@
 P 2700 4550
 AR Path="/5E2485D3" Ref="TP?"  Part="1"
-AR Path="/5E23D312/5E2485D3" Ref="B"  Part="1"
-F 0 "B" H 2673 4752 50  0000 L CNN
+AR Path="/5E23D312/5E2485D3" Ref="TP5"  Part="1"
+F 0 "TP5" H 2673 4752 50  0000 L CNN
 F 1 "TestPoint" H 2758 4577 50  0001 L CNN
 F 2 "" H 2900 4550 50  0001 C CNN
@@
 P 4200 4550
 AR Path="/5E248B58" Ref="TP?"  Part="1"
-AR Path="/5E23D312/5E248B58" Ref="C"  Part="1"
-F 0 "C" H 4174 4762 50  0000 L CNN
+AR Path="/5E23D312/5E248B58" Ref="TP9"  Part="1"
+F 0 "TP9" H 4174 4762 50  0000 L CNN
 F 1 "TestPoint" H 4258 4577 50  0001 L CNN
 F 2 "" H 4400 4550 50  0001 C CNN
@@
 P 4200 4950
 AR Path="/5E24914E" Ref="TP?"  Part="1"
-AR Path="/5E23D312/5E24914E" Ref="D"  Part="1"
-F 0 "D" H 4169 5163 50  0000 L CNN
+AR Path="/5E23D312/5E24914E" Ref="TP10"  Part="1"
+F 0 "TP10" H 4169 5163 50  0000 L CNN
 F 1 "TestPoint" H 4258 4977 50  0001 L CNN
 F 2 "" H 4400 4950 50  0001 C CNN
@@
 P 3300 4950
 AR Path="/5E2497A0" Ref="TP?"  Part="1"
-AR Path="/5E23D312/5E2497A0" Ref="E"  Part="1"
-F 0 "E" H 3273 5168 50  0000 L CNN
+AR Path="/5E23D312/5E2497A0" Ref="TP8"  Part="1"
+F 0 "TP8" H 3273 5168 50  0000 L CNN
 F 1 "TestPoint" H 3358 4977 50  0001 L CNN
 F 2 "" H 3500 4950 50  0001 C CNN
@@
 P 1950 4950
 AR Path="/5E249C9C" Ref="TP?"  Part="1"
-AR Path="/5E23D312/5E249C9C" Ref="F"  Part="1"
-F 0 "F" H 1921 5165 50  0000 L CNN
+AR Path="/5E23D312/5E249C9C" Ref="TP4"  Part="1"
+F 0 "TP4" H 1921 5165 50  0000 L CNN
 F 1 "TestPoint" H 2008 4977 50  0001 L CNN
 F 2 "" H 2150 4950 50  0001 C CNN
