File: S2020/file5E6D26B7.sch (KiCad schematic (older format))
At the start: 38 parts, among them SW1 SW_Push, U1 7404, U1 74LS32, U2 7404, U2 74LS08, U3 74LS08

Commit message: mess
Parts:
- gave numbers to parts that had none: 4
- renumbered Amp-Meter to Amp-Meter1, D1 to D32, D2 to D33, MES1 to MES2, R1 to R74, R2 to R75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
