File: S2020/opamps.sch (KiCad schematic (older format))
At the start: 44 parts, among them U1 LM741

Commit message: mess
Parts:
- gave numbers to parts that had none: 2
- renumbered BT to BT4, BT to BT5, D1 to D21, D2 to D22, R1 to R33, R1 to R34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
