File: S2020/stuff.sch (KiCad schematic (older format))
At the start: 37 parts

Commit message: mess
Parts:
- added D?: Error, symbol 00TJR:LED_small
- added D?: LED_small, symbol 00TJR:LED_small
- added R, R?: 330Ω, symbol Device:R_US
- added RN?: R_10k_SIPx08, Resistor_THT:R_Array_SIP9, symbol Device:R_Network08_US
- added SW?: SW_DIP_x08, symbol Switch:SW_DIP_x08
- added TTL: 10Hz, symbol 00TJR:SQgen
- added U? (x9): 74LS08, symbol 74xx:74LS08
- added U?: 74LS04, symbol 74xx:74LS04
- added U? (x18): 74LS86, symbol 74xx:74LS86
- added U? (x5): 74LS32, symbol 74xx:74LS32
- RN2: renamed from RN?; value R_Pack08_US -> R_330_DIPx08
- gave numbers to parts that had none: 36
Connections:
- net VCC is gone; now on net +5V: U23.16 (VCC), U24.16 (VCC), U25.16 (VCC), U38.16 (VCC), U39.16 (VCC)
- net +5V: now also D34.2 (A), D35.2 (A), D36.2 (A), D37.2 (A), D38.2 (A), D39.2 (A), D40.2 (A), D41.2 (A), D?.2 (A), D?.2 (A), RN?.1 (common)
- net A: now also U?.1, U?.1, U?.1, U?.1, U?.1, U?.1, U?.1, U?.1, U?.1, U?.2, U?.2, U?.2, U?.2, U?.2
- net B: now also U?.1, U?.1, U?.1, U?.1, U?.1, U?.2, U?.2, U?.2, U?.2, U?.2, U?.2, U?.2, U?.2, U?.2
- net GND: now also U23.4 (~G2A), U23.5 (~G2B), U24.7 (~E), SW?.1, SW?.2, SW?.3, SW?.4, SW?.5, SW?.6, SW?.7, SW?.8, TTL.2
- net DEMUX_S0: now reaches U23.1 (A0)
- net DEMUX_S0: now also RN?.2 (R1), SW?.16, U?.1
- net at U23.10 (~Y5): now also RN2.11, U24.14 (I5)
- net at U23.11 (~Y4): now also RN2.12, U24.15 (I4)
- net at U23.12 (~Y3): now also RN2.13, U24.1 (I3)
- net at U23.13 (~Y2): now also RN2.14, U24.2 (I2)
- net at U23.14 (~Y1): now also RN2.15, U24.3 (I1)
- net at U23.15 (~Y0), U24.4 (I0): now also RN2.16
- net DEMUX_S1: now reaches U23.2 (A1)
- net DEMUX_S1: now also RN?.3 (R2), SW?.15, U?.2
- net DEMUX_S2: now reaches U23.3 (A2)
- net DEMUX_S2: now also RN?.4 (R3), SW?.14, U?.2
- net at U23.6 (G1): now also TTL.1
- net at U23.7 (~Y7): now also RN2.9, U24.12 (I7)
- net at U23.9 (~Y6): now also RN2.10, U24.13 (I6)
- net MUX_S1: now reaches U24.10 (S1)
- net MUX_S1: now also RN?.8 (R7), SW?.10, U?.2
- net MUX_S0: now reaches U24.11 (S0)
- net MUX_S0: now also RN?.7 (R6), SW?.11, U?.1
- net at U24.6 (~Q): now also R.2
- net MUX_S2: now reaches U24.9 (S2)
- net MUX_S2: now also RN?.9 (R8), SW?.9, U?.2
- net at RN2.1: now also D41.1 (K)
- net at RN2.2: now also D40.1 (K)
- net at RN2.3: now also D39.1 (K)
- net at RN2.4: now also D38.1 (K)
- net at RN2.5: now also D37.1 (K)
- net at RN2.6: now also D36.1 (K)
- net at RN2.7: now also D35.1 (K)
- net at RN2.8: now also D34.1 (K)
- new net: U?.2, U?.5
- new net: U?.1, U?.3 (x6)
- new net: RN?.5 (R4), SW?.13
- new net: RN?.6 (R5), SW?.12
- new net: U?.1, U?.2, U?.3 (x5)
- new net: R?.2, U?.3
- new net: D?.1 (K), R?.1
- new net: D?.1 (K), R.1
- new net: U?.2, U?.3 (x5)
- new net Address: U?.1, U?.2
- new net Cin: U?.1, U?.1
- new net Cout: U?.3, U?.3, U?.3, U?.3
- new net Data: U?.1, U?.4
- new net PARITY: U?.2, U?.3
- new net Y0: U?.6
- new net Y1: U?.3
- new net ∑: U?.3, U?.3, U?.3, U?.3, U?.3, U?.3, U?.3
- no-connect marks 0 -> 3
Other:
- note added: "DEMUX Select"
- note added: "Data In"
- note added: "Data Out"
- note added: "MUX Select"
- moved on the sheet: RN2, Temp1, U23, U24, U41
